File: Eagle/PL-N823-01 Analog Breakout.brd (EAGLE design)
At the start: 25.4 x 25.4 mm, 33 parts, among them U1 ADS1015, U2 LMV358, U3 PL-N823-01

Commit message: v1.5 file update
Parts:
- R1: value 1k -> 27
Connections:
- net SIGNAL: no longer R3.1, U3.SOURCE
- net SOURCE: now also R3.1, U3.SOURCE
Routing:
- net SOURCE: track 0.00 -> 12.8 mm
- net SIGNAL: track 26.3 -> 14.6 mm
Other:
- board text added: "v1.5"
- board text removed: "v1.3"
Changed lines of the file:
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@@
 <drawing>
 <settings>
-<setting alwaysvectorfont="yes"/>
+<setting alwaysvectorfont="no"/>
 <setting verticaltext="up"/>
 </settings>
@@
 <layers>
 <layer number="1" name="Top" color="4" fill="1" visible="no" active="yes"/>
-<layer number="16" name="Bottom" color="1" fill="1" visible="no" active="yes"/>
+<layer number="16" name="Bottom" color="1" fill="1" visible="yes" active="yes"/>
 <layer number="17" name="Pads" color="2" fill="1" visible="yes" active="yes"/>
 <layer number="18" name="Vias" color="2" fill="1" visible="yes" active="yes"/>
-<layer number="19" name="Unrouted" color="6" fill="1" visible="yes" active="yes"/>
+<layer number="19" name="Unrouted" color="6" fill="1" visible="no" active="yes"/>
 <layer number="20" name="Dimension" color="24" fill="1" visible="yes" active="yes"/>
 <layer number="21" name="tPlace" color="16" fill="1" visible="yes" active="yes"/>
@@
 <layer number="24" name="bOrigins" color="15" fill="1" visible="yes" active="yes"/>
 <layer number="25" name="tNames" color="10" fill="1" visible="no" active="yes"/>
-<layer number="26" name="bNames" color="7" fill="1" visible="no" active="yes"/>
-<layer number="27" name="tValues" color="10" fill="1" visible="no" active="yes"/>
+<layer number="26" name="bNames" color="7" fill="1" visible="yes" active="yes"/>
+<layer number="27" name="tValues" color="10" fill="1" visible="yes" active="yes"/>
 <layer number="28" name="bValues" color="7" fill="1" visible="no" active="yes"/>
 <layer number="29" name="tStop" color="7" fill="3" visible="no" active="yes"/>
@@
 <wire x1="25.4" y1="25.4" x2="25.4" y2="0" width="0.2032" layer="20"/>
 <wire x1="25.4" y1="0" x2="0" y2="0" width="0.1524" layer="20"/>
-<text x="19.685" y="3.683" size="0.9652" layer="16" font="vector" ratio="15" rot="MR0">v1.3</text>
+<text x="19.685" y="3.683" size="0.9652" layer="16" font="vector" ratio="15" rot="MR0">v1.5</text>
 <text x="24.13" y="5.08" size="0.6096" layer="16" font="vector" ratio="15" rot="MR0">JM</text>
 </plain>
@@
 <element name="FD2" library="SparkFun-Aesthetics" library_urn="urn:adsk.eagle:library:507" package="FIDUCIAL-MICRO" package3d_urn="urn:adsk.eagle:package:37111/1" value="FIDUCIALUFIDUCIAL" x="24.384" y="1.016" smashed="yes"/>
 <element name="U$8" library="buzzard_labels_pln82301" package="PL#N823#01_BREAKOUT0" value="" x="20.828" y="23.622" smashed="yes" rot="MR0"/>
-<element name="R1" library="SparkFun-Resistors" library_urn="urn:adsk.eagle:library:532" package="0603" package3d_urn="urn:adsk.eagle:package:39650/1" value="1k" x="22.6695" y="17.526" smashed="yes">
+<element name="R1" library="SparkFun-Resistors" library_urn="urn:adsk.eagle:library:532" package="0603" package3d_urn="urn:adsk.eagle:package:39650/1" value="27" x="22.6695" y="17.526" smashed="yes">
 <attribute name="NAME" x="20.2565" y="17.399" size="0.6096" layer="51"/>
-<attribute name="PROD_ID" value="RES-07856" x="22.6695" y="17.526" size="1.778" layer="27" display="off"/>
-<attribute name="VALUE" value="1k" x="22.098" y="16.4465" size="0.6096" layer="27"/>
+<attribute name="PROD_ID" value="RES-09334" x="22.6695" y="17.526" size="1.778" layer="27" display="off"/>
+<attribute name="VALUE" value="27" x="22.098" y="16.4465" size="0.6096" layer="27"/>
 </element>
 <element name="R6" library="SparkFun-Resistors" library_urn="urn:adsk.eagle:library:532" package="0603" package3d_urn="urn:adsk.eagle:package:39650/1" value="2.2k" x="16.5735" y="8.6995" smashed="yes" rot="R90">
@@
 </element>
 <element name="JP1" library="SparkFun-Jumpers" library_urn="urn:adsk.eagle:library:528" package="SMT-JUMPER_3_2-NC_TRACE_SILK" package3d_urn="urn:adsk.eagle:package:39289/1" value="JUMPER-SMT_3_2-NC_TRACE_SILK" x="12.573" y="8.5725" smashed="yes" rot="MR0">
-<attribute name="NAME" x="12.573" y="9.7155" size="0.6096" layer="26" font="vector" ratio="20" rot="MR0" align="bottom-center"/>
+<attribute name="NAME" x="12.573" y="9.7155" size="0.6096" layer="28" font="vector" ratio="20" rot="MR0" align="bottom-center"/>
 <attribute name="VALUE" x="12.573" y="7.4295" size="0.6096" layer="28" font="vector" ratio="20" rot="MR0" align="top-center"/>
 </element>
 <element name="JP2" library="SparkFun-Jumpers" library_urn="urn:adsk.eagle:library:528" package="SMT-JUMPER_2_NC_TRACE_SILK" package3d_urn="urn:adsk.eagle:package:39281/1" value="JUMPER-SMT_2_NC_TRACE_SILK" x="22.6695" y="19.7485" smashed="yes" rot="MR90">
-<attribute name="NAME" x="23.8125" y="19.7485" size="0.6096" layer="26" font="vector" ratio="20" rot="MR90" align="bottom-center"/>
+<attribute name="NAME" x="23.8125" y="19.7485" size="0.6096" layer="28" font="vector" ratio="20" rot="MR90" align="bottom-center"/>
 <attribute name="VALUE" x="22.7965" y="23.0505" size="0.6096" layer="28" font="vector" ratio="20" rot="MR180" align="top-center"/>
 </element>
@@
 <signal name="SOURCE">
 <contactref element="U2" pad="3"/>
+<contactref element="U3" pad="SOURCE"/>
+<contactref element="R3" pad="1"/>
+<wire x1="11.575" y1="14.5665" x2="11.575" y2="15.7" width="0.254" layer="1"/>
+<wire x1="11.575" y1="15.7" x2="12.025" y2="16.15" width="0.254" layer="1"/>
+<wire x1="12.9" y1="16.15" x2="13.335" y2="16.585" width="0.254" layer="1"/>
+<wire x1="13.335" y1="16.585" x2="13.335" y2="17.52" width="0.254" layer="1"/>
+<wire x1="12.025" y1="16.15" x2="12.9" y2="16.15" width="0.254" layer="1"/>
+<wire x1="17.184" y1="23.4315" x2="16.15" y2="23.4315" width="0.254" layer="1"/>
+<wire x1="16.15" y1="23.4315" x2="15.65" y2="22.9315" width="0.254" layer="1"/>
+<wire x1="15.65" y1="22.9315" x2="15.65" y2="21.45" width="0.254" layer="1"/>
+<wire x1="15.65" y1="21.45" x2="14.95" y2="20.75" width="0.254" layer="1"/>
+<wire x1="14.15" y1="20.75" x2="14.95" y2="20.75" width="0.254" layer="1"/>
+<wire x1="13.335" y1="19.935" x2="14.15" y2="20.75" width="0.254" layer="1"/>
+<wire x1="13.335" y1="17.52" x2="13.335" y2="19.935" width="0.254" layer="1"/>
 </signal>
 <signal name="SIGNAL">
 <contactref element="U2" pad="1"/>
 <contactref element="R4" pad="2"/>
-<contactref element="U3" pad="SOURCE"/>
-<contactref element="R3" pad="1"/>
 <contactref element="U1" pad="4"/>
-<wire x1="10.795" y1="17.52" x2="10.795" y2="19.685" width="0.2032" layer="1"/>
-<wire x1="14.9225" y1="21.9075" x2="16.4465" y2="23.4315" width="0.2032" layer="1"/>
-<wire x1="16.4465" y1="23.4315" x2="17.184" y2="23.4315" width="0.2032" layer="1"/>
-<wire x1="10.795" y1="19.685" x2="13.0175" y2="21.9075" width="0.2032" layer="1"/>
-<wire x1="13.0175" y1="21.9075" x2="14.9225" y2="21.9075" width="0.2032" layer="1"/>
-<wire x1="11.575" y1="14.5665" x2="11.575" y2="15.73" width="0.2032" layer="1"/>
-<wire x1="10.795" y1="16.51" x2="10.795" y2="17.52" width="0.2032" layer="1"/>
-<wire x1="11.575" y1="15.73" x2="10.795" y2="16.51" width="0.2032" layer="1"/>
+<wire x1="10.795" y1="17.52" x2="10.795" y2="18.885" width="0.2032" layer="1"/>
 <wire x1="10.795" y1="17.52" x2="10.7375" y2="17.4625" width="0.2032" layer="1"/>
 <wire x1="10.7375" y1="17.4625" x2="10.16" y2="17.4625" width="0.2032" layer="1"/>
@@
 <wire x1="5.3975" y1="22.86" x2="7.3025" y2="22.86" width="0.2032" layer="1"/>
 <wire x1="8.5725" y1="21.59" x2="8.5725" y2="20.0025" width="0.2032" layer="1"/>
-<wire x1="8.5725" y1="20.0025" x2="8.89" y2="19.685" width="0.2032" layer="1"/>
+<wire x1="8.89" y1="19.685" x2="8.5725" y2="20.0025" width="0.2032" layer="1"/>
 <wire x1="7.3025" y1="22.86" x2="8.5725" y2="21.59" width="0.2032" layer="1"/>
-<wire x1="8.89" y1="19.685" x2="10.795" y2="19.685" width="0.2032" layer="1"/>
+<wire x1="10.795" y1="18.885" x2="9.995" y2="19.685" width="0.2" layer="1"/>
+<wire x1="9.995" y1="19.685" x2="8.89" y2="19.685" width="0.2" layer="1"/>
 </signal>
 <signal name="SDA">
