File: Eagle/PL-N823-01 Analog Breakout.sch (EAGLE design)
At the start: 22 parts, among them U1 ADS1015, U2 LMV358, U3 PL-N823-01

Commit message: v1.5 file update
Parts:
- R1: value 1k -> 27; device SparkFun-Resistors:1KOHM-0603-1/10W-1% -> SparkFun-Resistors:27OHM-0603-1/10W-1%
Connections:
- net SIGNAL: no longer R3.1, U3.SOURCE
- net SOURCE: now also R3.1, U3.SOURCE
Other:
- note added: "1.5"
- note removed: "1.2"
Changed lines of the file:
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@@
 <part name="FD1" library="SparkFun-Aesthetics" library_urn="urn:adsk.eagle:library:507" deviceset="FIDUCIAL" device="UFIDUCIAL" package3d_urn="urn:adsk.eagle:package:37111/1"/>
 <part name="FD2" library="SparkFun-Aesthetics" library_urn="urn:adsk.eagle:library:507" deviceset="FIDUCIAL" device="UFIDUCIAL" package3d_urn="urn:adsk.eagle:package:37111/1"/>
-<part name="R1" library="SparkFun-Resistors" library_urn="urn:adsk.eagle:library:532" deviceset="1KOHM" device="-0603-1/10W-1%" package3d_urn="urn:adsk.eagle:package:39650/1" value="1k"/>
+<part name="R1" library="SparkFun-Resistors" library_urn="urn:adsk.eagle:library:532" deviceset="27OHM" device="-0603-1/10W-1%" package3d_urn="urn:adsk.eagle:package:39650/1" value="27"/>
 <part name="GND6" library="SparkFun-PowerSymbols" library_urn="urn:adsk.eagle:library:530" deviceset="GND" device=""/>
 <part name="R6" library="SparkFun-Resistors" library_urn="urn:adsk.eagle:library:532" deviceset="2.2KOHM" device="-0603-1/10W-1%" package3d_urn="urn:adsk.eagle:package:39650/1" value="2.2k"/>
@@
 <text x="15.24" y="86.36" size="3.81" layer="150">Analog signal amplifier</text>
 <text x="167.64" y="11.43" size="2.54" layer="94">Brandon Williams</text>
-<text x="238.76" y="7.62" size="2.54" layer="94">1.2</text>
+<text x="238.76" y="7.62" size="2.54" layer="94">1.5</text>
 <wire x1="111.76" y1="160.02" x2="152.4" y2="160.02" width="0.1524" layer="97" style="longdash"/>
 <wire x1="152.4" y1="160.02" x2="152.4" y2="185.42" width="0.1524" layer="97" style="longdash"/>
@@
 <pinref part="U2" gate="G1" pin="+IN"/>
 <wire x1="33.02" y1="68.58" x2="30.48" y2="68.58" width="0.1524" layer="91"/>
-<wire x1="30.48" y1="68.58" x2="30.48" y2="76.2" width="0.1524" layer="91"/>
-<label x="30.48" y="76.2" size="1.778" layer="95"/>
-</segment>
-</net>
-<net name="SIGNAL" class="0">
-<segment>
-<label x="53.34" y="66.04" size="1.778" layer="95"/>
-<wire x1="48.26" y1="66.04" x2="50.8" y2="66.04" width="0.1524" layer="91"/>
-<pinref part="U2" gate="G1" pin="OUT"/>
-<pinref part="R4" gate="G$1" pin="2"/>
-<wire x1="50.8" y1="66.04" x2="53.34" y2="66.04" width="0.1524" layer="91"/>
-<wire x1="50.8" y1="55.88" x2="50.8" y2="66.04" width="0.1524" layer="91"/>
-<junction x="50.8" y="66.04"/>
+<label x="30.48" y="68.58" size="1.27" layer="95" rot="R180" xref="yes"/>
 </segment>
 <segment>
@@
 <label x="53.34" y="152.4" size="1.27" layer="95" xref="yes"/>
 </segment>
-<segment>
+</net>
+<net name="SIGNAL" class="0">
+<segment>
+<wire x1="48.26" y1="66.04" x2="50.8" y2="66.04" width="0.1524" layer="91"/>
+<pinref part="U2" gate="G1" pin="OUT"/>
+<pinref part="R4" gate="G$1" pin="2"/>
+<wire x1="50.8" y1="66.04" x2="53.34" y2="66.04" width="0.1524" layer="91"/>
+<wire x1="50.8" y1="55.88" x2="50.8" y2="66.04" width="0.1524" layer="91"/>
+<junction x="50.8" y="66.04"/>
+<label x="53.34" y="66.04" size="1.27" layer="95" xref="yes"/>
+</segment>
+<segment>
